File: Spaceport/PCBs/STM32 Flight Computer/STM32_Flight_Computer/STM32_Flight_Computer.kicad_sch (KiCad schematic)
At the start: 7 parts, among them IC1 ESP32-H2-MINI-1-N4, J1 USB4105-GF-A-060, U1 BMI088, U2 DPS368XTSA1, U3 LIS3MDLTR, U4 SAM-M8Q, U5 STM32H7A3ZIT6

Commit message: Schematic Hierarchy
- Added a page for reach sensor for better organization
Parts:
- removed IC1: ESP32-H2-MINI-1-N4, ESP32H2MINI1N4, symbol SRAD_AVIONICS:ESP32-H2-MINI-1-N4
- removed J1: USB4105-GF-A-060, USB4105-GF-A-060:GCT_USB4105-GF-A-060, symbol SRAD_AVIONICS:USB4105-GF-A-060
- removed U1: BMI088, BMI088:PQFN50P450X300X100-16N, symbol SRAD_AVIONICS:BMI088
- removed U2: DPS368XTSA1, DPS368XTSA1:XDCR_DPS368XTSA1, symbol SRAD_AVIONICS:DPS368XTSA1
- removed U3: LIS3MDLTR, LGA-12_2X2X1_STM, symbol SRAD_AVIONICS:LIS3MDLTR
- removed U4: SAM-M8Q, QFN_M-M8Q_UBL, symbol SRAD_AVIONICS:SAM-M8Q
- added H1, H2, H3, H4: MountingHole, MountingHole:MountingHole_3.2mm_M3, symbol Mechanical:MountingHole
Other:
- added sheet BT (BT.kicad_sch)
- added sheet Barometer (Barometer.kicad_sch)
- added sheet GPS (GPS.kicad_sch)
- added sheet IMU (IMU.kicad_sch)
- added sheet Magnometer (Magnometer.kicad_sch)
- added sheet USB_C (USB_C.kicad_sch)
- note added: "Mounting Holes"
- note added: "SENSORS"
