File: Spaceport/PCBs/STM32 Flight Computer/STM32_Flight_Computer/STM32_Flight_Computer.kicad_sch (KiCad schematic)
At the start: 5 parts, among them U5 STM32H7A3ZIT6

Commit message: Subcircuit Updates
Other:
- sheet IMU renamed IMU_24g
- removed sheet BT
- added sheet IMU_400g (IMU_400g.kicad_sch)
- added sheet LoRa_RFIC (LoRa_RFIC.kicad_sch)
Changed lines of the file:
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@@
 	)
 	(rectangle
-		(start -102.87 172.72)
-		(end -3.81 19.05)
+		(start 303.53 19.05)
+		(end 401.32 175.26)
+		(stroke
+			(width 0.3)
+			(type dash)
+		)
+		(fill
+			(type none)
+		)
+	)
+	(rectangle
+		(start -102.87 19.05)
+		(end -3.81 175.26)
 		(stroke
 			(width 0.3)
@@
 			)
 			(justify left)
+		)
+	)
+	(text "SENSORS"
+		(exclude_from_sim no)
+		(at 358.394 12.7 0)
+		(effects
+			(font
+				(face "Consolas")
+				(size 3 3)
+				(thickness 1)
+				(bold yes)
+			)
+			(justify right)
 		)
 	)
@@
 	)
 	(sheet
-		(at -49.53 74.93)
+		(at -50.8 124.46)
 		(size 39.37 44.45)
 		(fields_autoplaced yes)
@@
 		)
 		(property "Sheetname" "Barometer"
-			(at -49.53 74.2184 0)
+			(at -50.8 123.7484 0)
 			(effects
 				(font
@@
 		)
 		(property "Sheetfile" "Barometer.kicad_sch"
-			(at -49.53 119.9646 0)
+			(at -50.8 169.4946 0)
 			(effects
 				(font
@@
 			(color 0 0 0 0.0000)
 		)
-		(property "Sheetname" "IMU"
+		(property "Sheetname" "IMU_24g"
 			(at -96.52 74.2184 0)
 			(effects
@@
 	)
 	(sheet
-		(at -49.53 124.46)
+		(at -96.52 124.46)
 		(size 39.37 44.45)
 		(fields_autoplaced yes)
@@
 			(color 0 0 0 0.0000)
 		)
-		(property "Sheetname" "BT"
-			(at -49.53 123.7484 0)
+		(property "Sheetname" "USB_C"
+			(at -96.52 123.7484 0)
 			(effects
 				(font
@@
 			)
 		)
-		(property "Sheetfile" "BT.kicad_sch"
-			(at -49.53 169.4946 0)
+		(property "Sheetfile" "USB_C.kicad_sch"
+			(at -96.52 169.4946 0)
 			(effects
 				(font
@@
 			(project "STM32_Flight_Computer"
 				(path "/0f7e02ee-5e4c-4ec0-84f8-a7bba184df93"
-					(page "6")
+					(page "5")
 				)
 			)
@@
 	)
 	(sheet
-		(at -96.52 124.46)
+		(at 308.61 24.13)
 		(size 39.37 44.45)
 		(fields_autoplaced yes)
@@
 			(color 0 0 0 0.0000)
 		)
-		(property "Sheetname" "USB_C"
-			(at -96.52 123.7484 0)
+		(property "Sheetname" "LoRa_RFIC"
+			(at 308.61 23.4184 0)
 			(effects
 				(font
@@
 			)
 		)
-		(property "Sheetfile" "USB_C.kicad_sch"
-			(at -96.52 169.4946 0)
+		(property "Sheetfile" "LoRa_RFIC.kicad_sch"
+			(at 308.61 69.1646 0)
 			(effects
 				(font
@@
 			(project "STM32_Flight_Computer"
 				(path "/0f7e02ee-5e4c-4ec0-84f8-a7bba184df93"
-					(page "5")
-				)
-			)
+					(page "8")
+				)
+			)
+		)
+	)
+	(sheet
+		(at -50.8 74.93)
+		(size 39.37 44.45)
+		(fields_autoplaced yes)
+		(stroke
+			(width 0.1524)
+			(type solid)
+		)
+		(fill
+			(color 0 0 0 0.0000)
+		)
+		(property "Sheetname" "IMU_400g"
+			(at -50.8 74.2184 0)
+			(effects
+				(font
+					(size 1.27 1.27)
+				)
+				(justify left bottom)
+			)
+		)
+		(property "Sheetfile" "IMU_400g.kicad_sch"
+			(at -50.8 119.9646 0)
+			(effects
+				(font
+					(size 1.27 1.27)
+				)
+				(justify left top)
+			)
+		)
+		(instances
+			(project "STM32_Flight_Computer"
+				(path "/0f7e02ee-5e4c-4ec0-84f8-a7bba184df93"
+					(page "6")
+				)
+			)

Commit message: Push
Other:
- note added: "RF"
Changed lines of the file:
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@@
 		)
 	)
-	(text "SENSORS"
+	(text "RF"
 		(exclude_from_sim no)
 		(at 358.394 12.7 0)

Commit message: Push
Parts:
- added U9: W25N02KVZEIR, SON_WSON8_ZE_WIN, symbol SRAD_AVIONICS:W25N02KVZEIR
Connections:
- new net +3.3V: U9.8 (VSS)
- new net GND: U9.4 (GND), U9.9 (EPAD)
- new net PE11: U9.1 (/CS)
- new net PE2: U9.3 (/WP_(IO2))
- new net PF10: U9.6 (CLK)
- new net PF6: U9.7 (/HOLD_(IO3))
- new net PF8: U9.5 (DI_(IO0))
- new net PF9: U9.2 (DO_(IO1))
Other:
- moved on the sheet: U5A

Commit message: Push after Schematic Review 5/5
- Updated STM32 symbol
- Configured I2C busses
- Updated DC caps to 100nF
- TODO add power system things
Parts:
- removed U5: STM32H7A3ZIT6, LQFP-144, symbol SRAD_AVIONICS:STM32H7A3ZIT6
- added C15: 100nF, symbol Device:C
- added U5: STM32H7A3ZITx, Package_QFP:LQFP-144_20x20mm_P0.5mm, symbol MCU_ST_STM32H7:STM32H7A3ZITx
Connections:
- net +3.3V: now also C15.2
- net GND: now also C15.1
- net PE11: now also U5.64 (PE11)
- net PE2: now also U5.1 (PE2)
- net PF10: now also U5.22 (PF10)
- net PF6: now also U5.18 (PF6)
- net PF8: now also U5.20 (PF8)
- net PF9: now also U5.21 (PF9)
- new net: U5.107 (VSS), U5.120 (VSS), U5.130 (VSS), U5.16 (VSS), U5.38 (VSS), U5.51 (VSS), U5.61 (VSS), U5.83 (VSS), U5.94 (VSS)
Other:
- note added: "I2C1"
- note added: "I2C2"
- moved on the sheet: H1, H2, H3, H4, U9

Commit message: Push
Parts:
- removed U9: W25N02KVZEIR, SON_WSON8_ZE_WIN, symbol SRAD_AVIONICS:W25N02KVZEIR
- added C16: 100nF, symbol Device:C
- added C17: C, symbol Device:C
- added U10: MX25R6435FM2IL0, SOP_8L_200_MAC, symbol SRAD_AVIONICS:MX25R6435FM2IL0
- C15: value 100nF -> C
Connections:
- net +3.3V: now also U5.108 (VDD), U5.121 (VDDMMC), U5.131 (VDD), U5.144 (VDD), U5.17 (VDD), U5.30 (VDD), U5.33 (VDDA), U5.39 (VDD), U5.52 (VDD), U5.6 (VBAT), U5.62 (VDD), U5.72 (VDD), U5.84 (VDD), U5.95 (VDD33_USB), C16.2, U10.8 (VCC); no longer C15.2
- net GND: now also C15.2, U5.107 (VSS), U5.120 (VSS), U5.130 (VSS), U5.16 (VSS), U5.31 (VSSA), U5.38 (VSS), U5.51 (VSS), U5.61 (VSS), U5.83 (VSS), U5.94 (VSS), C16.1, C17.2, U10.4 (GND); no longer C15.1
- net PE11: now also U10.1 (CS#)
- net PE2: now also U10.3 (WP#/SIO2)
- net PF10: now also U10.6 (SCLK)
- net PF6: now also U10.7 (RESET#/SIO3)
- net PF8: now also U10.5 (SI/SIO0)
- net PF9: now also U10.2 (SO/SIO1)
- net SCL1: now also U5.136 (PB6)
- net SCL2: now also U5.11 (PF1)
- net SDA1: now also U5.137 (PB7)
- net SDA2: now also U5.10 (PF0)
- net PA11: now reaches U5.103 (PA11)
- net PA12: now reaches U5.104 (PA12)
- net at U5.106 (VCAP): now also C15.1
- net PD7: now reaches U5.123 (PD7)
- net PG9: now reaches U5.124 (PG9)
- net PA0: now reaches U5.34 (PA0)
- net PA1: now reaches U5.35 (PA1)
- net PA2: now reaches U5.36 (PA2)
- net PA3: now reaches U5.37 (PA3)
- net PA4: now reaches U5.40 (PA4)
- net PA5: now reaches U5.41 (PA5)
- net at U5.71 (VCAP): now also C17.1
Other:
- added sheet Power (Power.kicad_sch)
- note added: "LoRa DIO8"
- note added: "LoRa DIO9"
- note added: "LoRa LR Busy"
- note added: "LoRa LR NRST"
- note added: "QSPI1"
- note added: "SPI1"
- note added: "USB OTG 1"
