File: Spaceport/PCBs/STM32 Flight Computer/STM32_Flight_Computer/BT.kicad_sch (KiCad schematic)
At the start: 1 part, among them IC1 ESP32-H2-MINI-1-N4

Commit message: Subcircuit Updates
Connections:
- net GND: now reaches IC1.36 (GND_5)
- net GND: now also IC1.37 (GND_6), IC1.38 (GND_7), IC1.39 (GND_8), IC1.40 (GND_9), IC1.41 (GND_10), IC1.42 (GND_11), IC1.43 (GND_12), IC1.44 (GND_13), IC1.45 (GND_14), IC1.46 (GND_15), IC1.47 (GND_16), IC1.48 (GND_17), IC1.49 (GND_18), IC1.50 (GND_19), IC1.51 (GND_20), IC1.52 (GND_21), IC1.53 (GND_22), IC1.54 (GND_23), IC1.55 (GND_24), IC1.56 (GND_25), IC1.57 (GND_26), IC1.58 (GND_27), IC1.59 (GND_28), IC1.60 (GND_29), IC1.61 (GND_30)
- no-connect marks 0 -> 4
