File: Spaceport/PCBs/STM32 Flight Computer/STM32_Flight_Computer/Barometer.kicad_sch (KiCad schematic)
At the start: 1 part, among them U2 DPS368XTSA1

Commit message: Subcircuit Updates
Parts:
- added C3, C4: 100nF, symbol Device:C
Connections:
- net GND: now reaches U2.1 (GND)
- net GND: now also U2.7 (GND__1), C3.2, C4.1
- net SDA0: now reaches U2.3 (SDI)
- net SCL0: now reaches U2.4 (SCK)
- net +3.3V: now reaches U2.6 (VDDIO)
- net +3.3V: now also U2.8 (VDD), C3.1, C4.2
- no-connect marks 0 -> 2
Other:
- moved on the sheet: U2

Commit message: Push after Schematic Review 5/5
- Updated STM32 symbol
- Configured I2C busses
- Updated DC caps to 100nF
- TODO add power system things
Connections:
- net GND: now also U2.5 (SDO)
- net SCL0 renamed SCL2
- net SDA0 renamed SDA2
- no-connect marks 2 -> 1
Other:
- note added: "0x76"
Changed lines of the file:
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@@
 		(at 128.27 90.17)
 	)
-	(no_connect
-		(at 128.27 97.79)
-	)
 	(wire
 		(pts
@@
 		)
 	)
-	(global_label "SDA0"
-		(shape input)
-		(at 128.27 95.25 180)
-		(fields_autoplaced yes)
+	(text "0x76"
+		(exclude_from_sim no)
+		(at 130.048 99.314 0)
 		(effects
 			(font
 				(size 1.27 1.27)
 			)
+		)
+	)
+	(global_label "SDA2"
+		(shape input)
+		(at 128.27 95.25 180)
+		(fields_autoplaced yes)
+		(effects
+			(font
+				(size 1.27 1.27)
+			)
 			(justify right)
 		)
@@
 		)
 	)
-	(global_label "SCL0"
+	(global_label "SCL2"
 		(shape input)
 		(at 128.27 92.71 180)
@@
 					(unit 1)
 				)
+			)
+		)
+	)
+	(symbol
+		(lib_id "power:GND")
+		(at 128.27 97.79 270)
+		(unit 1)
+		(exclude_from_sim no)
+		(in_bom yes)
+		(on_board yes)
+		(dnp no)
+		(fields_autoplaced yes)
+		(property "Reference" "#PWR080"
+			(at 121.92 97.79 0)
+			(effects
+				(font
+					(size 1.27 1.27)
+				)
+				(hide yes)
+			)
+		)
+		(property "Value" "GND"
+			(at 124.46 97.7899 90)
+			(effects
+				(font
+					(size 1.27 1.27)
+				)
+				(justify right)
+			)
+		)
+		(property "Footprint" ""
+			(at 128.27 97.79 0)
+			(effects
+				(font
+					(size 1.27 1.27)
+				)
+				(hide yes)
+			)
+		)
+		(property "Datasheet" ""
+			(at 128.27 97.79 0)
+			(effects
+				(font
+					(size 1.27 1.27)
+				)
+				(hide yes)
+			)
+		)
+		(property "Description" "Power symbol creates a global label with name \"GND\" , ground"
+			(at 128.27 97.79 0)
+			(effects
+				(font
+					(size 1.27 1.27)
+				)
+				(hide yes)
+			)
+		)
+		(pin "1"
+		)
+		(instances
+			(project "STM32_Flight_Computer"
+				(path "/0f7e02ee-5e4c-4ec0-84f8-a7bba184df93/6385d2e5-860d-4872-95dc-7fa1940dbd05"
+					(reference "#PWR080")
+					(unit 1)
+				)
