File: Spaceport/PCBs/STM32 Flight Computer/STM32_Flight_Computer/Magnometer.kicad_sch (KiCad schematic)
At the start: 1 part, among them U3 LIS3MDLTR

Commit message: Subcircuit Updates
Other:
- moved on the sheet: U3
Changed lines of the file:
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@@
 	(symbol
 		(lib_id "SRAD_AVIONICS:LIS3MDLTR")
-		(at 118.11 72.39 0)
+		(at 113.03 96.52 0)
 		(unit 1)
 		(exclude_from_sim no)
@@
 		(fields_autoplaced yes)
 		(property "Reference" "U3"
-			(at 148.59 62.23 0)
+			(at 143.51 86.36 0)
 			(effects
 				(font
@@
 		)
 		(property "Value" "LIS3MDLTR"
-			(at 148.59 64.77 0)
+			(at 143.51 88.9 0)
 			(effects
 				(font
@@
 		)
 		(property "Footprint" "LGA-12_2X2X1_STM"
-			(at 118.11 72.39 0)
+			(at 113.03 96.52 0)
 			(effects
 				(font
@@
 		)
 		(property "Datasheet" "LIS3MDLTR"
-			(at 118.11 72.39 0)
+			(at 113.03 96.52 0)
 			(effects
 				(font
@@
 		)
 		(property "Description" ""
-			(at 118.11 72.39 0)
+			(at 113.03 96.52 0)
 			(effects
 				(font

Commit message: Push
Parts:
- added C7, C9: 100nF, symbol Device:C
- added C8: 1uF, symbol Device:C
Connections:
- net SCL0: now reaches U3.1 (SCL/SPC)
- net +3.3V: now reaches U3.10 (CS)
- net +3.3V: now also U3.4 (C1), U3.5 (VDD), U3.6 (VDD_IO), C7.1, C9.1
- net SDA0: now reaches U3.11 (SDA/SDI/SDO)
- net GND: now reaches U3.12 (RES)
- net GND: now also U3.2 (RES), U3.3 (GND), C7.2, C8.1, C8.2, C9.2
- no-connect marks 0 -> 3

Commit message: Push after Schematic Review 5/5
- Updated STM32 symbol
- Configured I2C busses
- Updated DC caps to 100nF
- TODO add power system things
Parts:
- C8: value 1uF -> 100nF
Connections:
- net +3.3V: now also U3.9 (SDO/SA1)
- net SCL0 renamed SCL2
- net SDA0 renamed SDA2
- no-connect marks 3 -> 2
Other:
- note added: "0x1E"
Changed lines of the file:
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@@
+	)
+	(junction
+		(at 177.8 104.14)
+		(diameter 0)
+		(color 0 0 0 0)
 	)
 	(junction
@@
 		(diameter 0)
 		(color 0 0 0 0)
-	)
-	(no_connect
-		(at 173.99 104.14)
 	)
 	(no_connect
@@
 	(wire
 		(pts
-			(xy 177.8 118.11) (xy 177.8 101.6)
+			(xy 177.8 118.11) (xy 177.8 104.14)
 		)
 		(stroke
@@
 	(wire
 		(pts
+			(xy 173.99 104.14) (xy 177.8 104.14)
+		)
+		(stroke
+			(width 0)
+			(type default)
+		)
+	)
+	(wire
+		(pts
 			(xy 88.9 104.14) (xy 113.03 104.14)
 		)
@@
 	(wire
 		(pts
+			(xy 177.8 104.14) (xy 177.8 101.6)
+		)
+		(stroke
+			(width 0)
+			(type default)
+		)
+	)
+	(wire
+		(pts
 			(xy 91.44 101.6) (xy 91.44 106.68)
 		)
@@
 		)
 	)
-	(global_label "SDA0"
+	(text "0x1E"
+		(exclude_from_sim no)
+		(at 154.432 104.14 0)
+		(effects
+			(font
+				(size 1.27 1.27)
+			)
+		)
+	)
+	(global_label "SDA2"
 		(shape input)
 		(at 173.99 99.06 0)
@@
 		)
 	)
-	(global_label "SCL0"
+	(global_label "SCL2"
 		(shape input)
 		(at 113.03 96.52 180)
@@
 			)
 		)
-		(property "Value" "1uF"
+		(property "Value" "100nF"
 			(at 95.25 113.538 90)
 			(effects
