File: Spaceport/PCBs/STM32 Flight Computer/STM32_Flight_Computer/USB_C.kicad_sch (KiCad schematic)
At the start: 1 part, among them J1 USB4105-GF-A-060

Commit message: Subcircuit Updates
Parts:
- added U6: USBLC6-2P6, SRAD_AVIONICS:SOT-666_STM-L, symbol Power_Protection:USBLC6-2P6
Connections:
- net GND: now reaches J1.A1_B12 (GND)
- net GND: now also J1.A5 (CC1), J1.B1_A12 (GND__1), J1.SH1 (SHELL_GND), J1.SH2 (SHELL_GND__1), J1.SH3 (SHELL_GND__2), J1.SH4 (SHELL_GND__3), U6.2 (GND)
- net VBUS: now reaches J1.A4_B9 (VBUS)
- net VBUS: now also U6.5 (VBUS)
- net at J1.A6 (DP1): now also U6.1 (I/O1)
- net at J1.A7 (DN1): now also U6.3 (I/O2)
- new net DP1: U6.4 (I/O2), U6.6 (I/O1)
- no-connect marks 0 -> 6

Commit message: Push
Connections:
- net at J1.A6 (DP1), U6.1 (I/O1): now also J1.B6 (DP2)
- net at J1.A7 (DN1), U6.3 (I/O2): now also J1.B7 (DN2)
- no-connect marks 6 -> 4
Changed lines of the file:
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@@
+	)
+	(junction
+		(at 133.35 86.36)
+		(diameter 0)
+		(color 0 0 0 0)
 	)
 	(junction
@@
 	)
 	(junction
+		(at 133.35 83.82)
+		(diameter 0)
+		(color 0 0 0 0)
+	)
+	(junction
 		(at 181.61 99.06)
 		(diameter 0)
@@
 	)
 	(no_connect
-		(at 177.8 86.36)
-	)
-	(no_connect
 		(at 177.8 91.44)
 	)
@@
 	)
 	(no_connect
-		(at 177.8 88.9)
-	)
-	(no_connect
 		(at 177.8 78.74)
 	)
 	(wire
 		(pts
+			(xy 177.8 86.36) (xy 187.96 86.36)
+		)
+		(stroke
+			(width 0)
+			(type default)
+		)
+	)
+	(wire
+		(pts
 			(xy 181.61 106.68) (xy 181.61 104.14)
 		)
@@
 	(wire
 		(pts
-			(xy 129.54 83.82) (xy 137.16 83.82)
+			(xy 129.54 83.82) (xy 133.35 83.82)
 		)
 		(stroke
@@
 	(wire
 		(pts
-			(xy 129.54 86.36) (xy 137.16 86.36)
+			(xy 133.35 116.84) (xy 133.35 86.36)
+		)
+		(stroke
+			(width 0)
+			(type default)
+		)
+	)
+	(wire
+		(pts
+			(xy 133.35 67.31) (xy 133.35 83.82)
+		)
+		(stroke
+			(width 0)
+			(type default)
+		)
+	)
+	(wire
+		(pts
+			(xy 129.54 86.36) (xy 133.35 86.36)
 		)
 		(stroke
@@
 	(wire
 		(pts
+			(xy 177.8 88.9) (xy 187.96 88.9)
+		)
+		(stroke
+			(width 0)
+			(type default)
+		)
+	)
+	(wire
+		(pts
+			(xy 133.35 86.36) (xy 137.16 86.36)
+		)
+		(stroke
+			(width 0)
+			(type default)
+		)
+	)
+	(wire
+		(pts
 			(xy 177.8 99.06) (xy 181.61 99.06)
 		)
@@
 	(wire
 		(pts
+			(xy 133.35 83.82) (xy 137.16 83.82)
+		)
+		(stroke
+			(width 0)
+			(type default)
+		)
+	)
+	(wire
+		(pts
 			(xy 177.8 109.22) (xy 181.61 109.22)
 		)
@@
 	(wire
 		(pts
+			(xy 187.96 116.84) (xy 133.35 116.84)
+		)
+		(stroke
+			(width 0)
+			(type default)
+		)
+	)
+	(wire
+		(pts
+			(xy 187.96 67.31) (xy 133.35 67.31)
+		)
+		(stroke
+			(width 0)
+			(type default)
+		)
+	)
+	(wire
+		(pts
 			(xy 181.61 104.14) (xy 181.61 101.6)
 		)
@@
 	(wire
 		(pts
+			(xy 187.96 88.9) (xy 187.96 116.84)
+		)
+		(stroke
+			(width 0)
+			(type default)
+		)
+	)
+	(wire
+		(pts
 			(xy 181.61 99.06) (xy 181.61 96.52)
 		)
@@
 		)
 		(stroke
+			(width 0)
+			(type default)
+		)
+	)
+	(wire
+		(pts
+			(xy 187.96 86.36) (xy 187.96 67.31)
+		)
+		(stroke

Commit message: Push after Schematic Review 5/5
- Updated STM32 symbol
- Configured I2C busses
- Updated DC caps to 100nF
- TODO add power system things
Parts:
- added R2, R3: 5.1k, symbol Device:R
Connections:
- net DP1: now also J1.A6 (DP1), J1.B6 (DP2), U6.1 (I/O1); no longer U6.4 (I/O2), U6.6 (I/O1)
- net GND: now also R2.1, R3.2; no longer J1.A5 (CC1)
- net VBUS: now also J1.B4_A9 (VBUS__1)
- net DN1: now reaches J1.A7 (DN1), J1.B7 (DN2), U6.3 (I/O2)
- net at J1.B5 (CC2): now also R3.1
- new net: J1.A5 (CC1), R2.2
- new net PA11: U6.4 (I/O2)
- new net PA12: U6.6 (I/O1)
- no-connect marks 4 -> 2
Other:
- moved on the sheet: U6

Commit message: Push
Other:
- note added: "+5V"
Changed lines of the file:
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@@
 (kicad_sch
-	(version 20231120)
+	(version 20250114)
 	(generator "eeschema")
-	(generator_version "8.0")
+	(generator_version "9.0")
 	(paper "A4")
+	(text "+5V"
+		(exclude_from_sim no)
+		(at 188.214 74.422 0)
+		(effects
+			(font
+				(size 1.27 1.27)
+			)
+		)
+	)
 	(junction
 		(at 181.61 101.6)
