File: Spaceport/PCBs/ESP32 Ground Station/ESP32 Ground Station.kicad_sch (KiCad schematic)
At the start: 49 parts, among them J1 Micro_SD_Card_Det1, J2 Conn_01x02, J3 USB_C_Receptacle_USB2.0_16P, J4 Conn_Coaxial, J7 Conn_01x10, J8 Conn_01x10, SW1 SW_SPST, U1 ESP32-S3-MINI-1, U2 LBAA0XV2GT-001, U3 XC6220B331MR, U4 USBLC6-2P6, U5 TPS22917DBV, U6 BQ25185DLHR

Commit message: early pcb layout
Parts:
- BZ1: footprint (none) -> Buzzer_Beeper:Buzzer_TDK_PS1240P02BT_D12.2mm_H6.5mm
- C1, C2, C3, C4, C7: footprint (none) -> Capacitor_SMD:C_0603_1608Metric
- C5, C6: value C -> DNP; footprint (none) -> Capacitor_SMD:C_0603_1608Metric
- D1, D2, D3, D6: footprint (none) -> LED_SMD:LED_0805_2012Metric
- D4, D5: footprint (none) -> Diode_SMD:D_0603_1608Metric
- J1: footprint (none) -> MEM2085:GCT_MEM2085-00-115-00-A_REV0.2
- J2: value Conn_01x02 -> BAT; footprint (none) -> Connector_JST:JST_PH_S2B-PH-K_1x02_P2.00mm_Horizontal
- J3: footprint (none) -> Connector_USB:USB_C_Receptacle_GCT_USB4105-xx-A_16P_TopMnt_Horizontal
- J4: value Conn_Coaxial -> SMA; footprint (none) -> Connector_Coaxial:SMA_Amphenol_132289_EdgeMount
- J7, J8: footprint (none) -> Connector_PinHeader_2.54mm:PinHeader_1x10_P2.54mm_Vertical
- L1: value L -> 0; footprint (none) -> Inductor_SMD:L_0603_1608Metric
- L2: footprint (none) -> Inductor_SMD:L_0603_1608Metric
- R1, R10, R11, R12, R13, R14, R15, R16, R17, R18, R19, R2, R20, R3, R4, R5, R6, R7, R8, R9: footprint (none) -> Resistor_SMD:R_0603_1608Metric
- SW1: footprint (none) -> 50-0118-00:50-0118-00
- U2: footprint LBAA0XV2GT001 -> Murata Radio:LBAA0XV2GT001
- U6: footprint WSON10_DLH_TEX -> footprints:WSON10_DLH_TEX
Connections:
- net BAT_MEAS: now also R19.2; no longer R19.1
- net VBAT: now also R19.1; no longer R19.2
Other:
- note added: "3.3v Linear Regulator"
- note added: "Battery Charger"
- note added: "ESD Protection"
- note added: "Power Switch"
- note added: "SMA Antenna"
- note added: "USB-C 2.0 Receptacle"
- note removed: "USB-C 2.0 Recepticle"
- moved on the sheet: R19, R20

Commit message: changes to GS layout and Schem
Parts:
- L2: footprint Inductor_SMD:L_0603_1608Metric -> Inductor_SMD:L_1210_3225Metric
Changed lines of the file:
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@@
 			)
 		)
-		(property "Footprint" "Inductor_SMD:L_0603_1608Metric"
+		(property "Footprint" "Inductor_SMD:L_1210_3225Metric"
 			(at 199.39 44.45 0)
 			(effects

Commit message: added data sheets to schematic
Other:
- note added: "Datasheet"
- note added: "Datasheet - LR1121"
- note added: "Datasheet - Switch"
Changed lines of the file:
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@@
+		)
+	)
+	(text "Datasheet"
+		(exclude_from_sim no)
+		(at 34.036 78.486 0)
+		(effects
+			(font
+				(size 1.27 1.27)
+			)
+			(href "https://mm.digikey.com/Volume0/opasdata/d220001/medias/docus/5702/USB4105%20-%20Product%20Drawing.pdf")
 		)
 	)
@@
 		)
 	)
+	(text "Datasheet"
+		(exclude_from_sim no)
+		(at 75.692 88.646 0)
+		(effects
+			(font
+				(size 1.27 1.27)
+			)
+			(href "https://www.st.com/content/ccc/resource/technical/document/datasheet/06/1d/48/9c/6c/20/4a/b2/CD00050750.pdf/files/CD00050750.pdf/jcr:content/translations/en.CD00050750.pdf")
+		)
+	)
+	(text "Datasheet"
+		(exclude_from_sim no)
+		(at 243.586 122.174 0)
+		(effects
+			(font
+				(size 1.27 1.27)
+			)
+			(href "https://mm.digikey.com/Volume0/opasdata/d220001/medias/docus/642/XC6220.pdf")
+		)
+	)
 	(text "Power Switch\n"
 		(exclude_from_sim no)
@@
 		)
 	)
+	(text "Datasheet"
+		(exclude_from_sim no)
+		(at 160.02 25.654 0)
+		(effects
+			(font
+				(size 1.27 1.27)
+			)
+			(href "https://www.espressif.com/sites/default/files/documentation/esp32-s3-mini-1_mini-1u_datasheet_en.pdf")
+		)
+	)
+	(text "Datasheet"
+		(exclude_from_sim no)
+		(at 82.804 27.432 0)
+		(effects
+			(font
+				(size 1.27 1.27)
+			)
+			(href "https://gct.co/files/drawings/mem2085.pdf")
+		)
+	)
 	(text "3.3v Linear Regulator"
 		(exclude_from_sim no)
@@
 		)
 	)
+	(text "Datasheet - Switch\n"
+		(exclude_from_sim no)
+		(at 207.01 110.998 0)
+		(effects
+			(font
+				(size 1.27 1.27)
+			)
+			(href "https://mm.digikey.com/Volume0/opasdata/d220001/medias/docus/5735/50-0118-00.pdf")
+		)
+	)
 	(text "ESD Protection\n"
 		(exclude_from_sim no)
@@
 		)
 	)
+	(text "Datasheet"
+		(exclude_from_sim no)
+		(at 200.152 26.416 0)
+		(effects
+			(font
+				(size 1.27 1.27)
+			)
+			(href "https://www.murata.com/-/media/webrenewal/products/connectivitymodule/lpwa/overview/lineup/pdf/type2gt.ashx?la=en-us&cvid=20240605010000000000")
+		)
+	)
+	(text "Datasheet"
+		(exclude_from_sim no)
+		(at 160.782 119.126 0)
+		(effects
+			(font
+				(size 1.27 1.27)
+			)
+			(href "https://www.ti.com/lit/ds/symlink/bq25185.pdf?ts=1701339761812&ref_url=https%253A%252F%252Fwww.ti.com%252Fproduct%252FBQ25185")
+		)
+	)
 	(text "Power and Batteries"
 		(exclude_from_sim no)
@@
 		)
 	)
+	(text "Datasheet"
+		(exclude_from_sim no)
+		(at 205.74 140.97 0)
+		(effects
+			(font
+				(size 1.27 1.27)
+			)
+			(href "https://www.ti.com/general/docs/suppproductinfo.tsp?distId=10&gotoUrl=https%3A%2F%2Fwww.ti.com%2Flit%2Fgpn%2Ftps22917")
+		)
+	)
+	(text "Datasheet - LR1121"
+		(exclude_from_sim no)
+		(at 226.568 26.416 0)
+		(effects
+			(font
+				(size 1.27 1.27)
+			)
+			(href "https://semtech.my.salesforce.com/sfc/p/#E0000000JelG/a/RQ0000093ZiP/RV4Ba6LROsFrFjnAAVK2av5W11RGmCms_3Q2cyKHdDA")
+		)
+	)

Commit message: add decoupling caps
Parts:
- removed L1: 0, Inductor_SMD:L_0603_1608Metric, symbol Device:L
- added C10, C11: 10u, Capacitor_SMD:C_0603_1608Metric, symbol Device:C
- added C8, C9: 100n, Capacitor_SMD:C_0603_1608Metric, symbol Device:C
- added R21: 0, Resistor_SMD:R_0603_1608Metric, symbol Device:R
Connections:
- net +3v3: now also C11.2, C8.1, C9.1
- net +4v5-2: now also C10.2
- net GND: now also C10.1, C11.1, C8.2, C9.2
- net at C6.1, J4.1 (In): now also R21.1
- net at C5.1, U2.19 (ANT_LORA_SUB_G_): now also R21.2
Other:
- moved on the sheet: R1
