File: Spaceport/PCBs/ESP32 Ground Station/ESP32 Ground Station.kicad_sch (KiCad schematic)
At the start: 50 parts, among them J1 Micro_SD_Card_Det1, J2 BAT, J3 USB_C_Receptacle_USB2.0_16P, J4 SMA, J5 Conn_02x10_Odd_Even, SW1 SW_SPST, U1 ESP32-S3-MINI-1, U2 LBAA0XV2GT-001, U3 XC6220B331MR, U4 USBLC6-2P6, U5 TPS22917DBV, U6 BQ25185DLHR

Commit message: GS Traces complete
Parts:
- added D7: PWR5, LED_SMD:LED_0805_2012Metric, symbol Device:LED
- added R22: 2k, Resistor_SMD:R_0603_1608Metric, symbol Device:R
- D3: value PWR -> PWR3
- J1: footprint MEM2085:GCT_MEM2085-00-115-00-A_REV0.2 -> MEM2085:microSD-GCT_MEM2085-00-115-00-A_REV0.2
Connections:
- net +3v3: no longer J1.5 (CLK), U1.5 (IO1)
- net GND: now also D7.1 (K)
- net VBUS: now also R22.2
- net DPWR renamed DPWR3
- new net DPWR5: D7.2 (A), R22.1
- new net SD_CLK: J1.5 (CLK), U1.5 (IO1)
