File: Spaceport/PCBs/ESP32 Ground Station/ESP32 Ground Station.kicad_pcb (KiCad board)
At the start: 2 copper layers, 39 x 49 mm, 49 parts, among them J1 Micro_SD_Card_Det1, J2 BAT, J3 USB_C_Receptacle_USB2.0_16P, J4 SMA, J7 Conn_01x10, J8 Conn_01x10, SW1 SW_SPST, U1 ESP32-S3-MINI-1, U2 LBAA0XV2GT-001, U3 XC6220B331MR, U4 USBLC6-2P6, U5 TPS22917DBV, U6 BQ25185DLHR

Commit message: changes to GS layout and Schem
Parts:
- J7, J8: moved to F.Cu
- L2: footprint Inductor_SMD:L_0603_1608Metric -> Inductor_SMD:L_1210_3225Metric
- moved R16 33.5 mm to (170.2, 83.0)
- moved R17 33.5 mm to (170.2, 85.5)
- moved R18 33.5 mm to (170.2, 88.0)
- moved R19 33.5 mm to (170.2, 90.5)
- moved R20 33.5 mm to (170.2, 93.0)
- moved C1 33.5 mm to (158.1, 83.0)
- moved C2 33.5 mm to (158.1, 85.5)
- moved C3 33.5 mm to (158.1, 88.0)
- moved C4 33.5 mm to (158.1, 90.5)
- moved C5 33.5 mm to (158.1, 93.0)
- moved C6 33.5 mm to (158.1, 95.5)
- moved C7 33.5 mm to (158.1, 98.0)
- moved L1 33.5 mm to (158.1, 100.5)
- moved L2 33.5 mm to (162.2, 83.0)
- moved R1 33.5 mm to (162.2, 85.5)
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
Commit message: Layout mostly done for GS
Parts:
- removed J7, J8: Conn_01x10, Connector_PinHeader_2.54mm:PinHeader_1x10_P2.54mm_Vertical
- removed L1: 0, Inductor_SMD:L_0603_1608Metric
- removed R9: 10k, Resistor_SMD:R_0603_1608Metric
- added C10: 10u, Capacitor_SMD:C_0603_1608Metric, B.Cu at (218.5, 101.5)
- added C11: 10u, Capacitor_SMD:C_0603_1608Metric, B.Cu at (222.0, 104.5)
- added C8: 100n, Capacitor_SMD:C_0603_1608Metric, F.Cu at (226.8, 109.3)
- added J5: Conn_02x10_Odd_Even, Connector_PinHeader_2.54mm:PinHeader_2x10_P2.54mm_Vertical, F.Cu at (200.0, 78.0)
- added R21: 0, Resistor_SMD:R_0603_1608Metric, F.Cu at (228.2, 104.3)
- BZ1, J2, J3, J4, SW1, U2: moved to F.Cu
- C1, C2, C3, C4, D4, D5, J1, R1, R10, R11, R12, R14, R19, R2, R20, R3, R4, R5, R6, R7, R8, U1, U3, U4, U5, U6: moved to B.Cu
- moved C6 72.1 mm to (229.8, 104.3), turned to -90 degrees
- moved R3 70.3 mm to (231.0, 76.5), turned to 90 degrees
- moved R4 69.6 mm to (231.0, 83.0), turned to -90 degrees
- moved C5 69.5 mm to (226.8, 104.3), turned to 90 degrees
- moved R6 61.1 mm to (222.0, 85.7), turned to 90 degrees
- moved R7 58.3 mm to (219.5, 89.8), turned to 180 degrees
- moved R13 57.2 mm to (221.5, 81.0)
- moved C4 57.1 mm to (215.0, 96.0), turned to 180 degrees
- moved C2 54.8 mm to (210.5, 101.5), turned to 90 degrees
- moved C7 54.7 mm to (211.8, 108.8), turned to -90 degrees
- moved L2 54.2 mm to (211.8, 104.8), turned to 90 degrees
- moved R8 54.0 mm to (219.5, 91.3), turned to 180 degrees
- moved C1 54.0 mm to (210.5, 96.0), turned to 180 degrees
- moved R10 53.7 mm to (219.5, 94.3), turned to 180 degrees
- moved R11 53.6 mm to (219.5, 95.8), turned to 180 degrees
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Connections:
- net Net-(D1-K) renamed /DSTAT1
- net Net-(D2-A) renamed /DSTAT2
- net Net-(D3-A) renamed /DPWR
- net Net-(D6-A) renamed /DGPIO
- net Net-(J3-CC1) renamed /CC1
- net Net-(J3-CC2) renamed /CC2
- net Net-(J3-D+-PadA6) renamed /D+_1
- net Net-(J3-D--PadA7) renamed /D-_1
- net Net-(J4-In) renamed /ANT_1
- net Net-(U2-ANT_LORA_SUB_G_) renamed /ANT
- net Net-(U2-DCC_SW) renamed /DCC
- net Net-(U2-VREG) renamed /VREG
- net Net-(U6-ILIM/VSET) renamed /ILIM
- net Net-(U6-ISET) renamed /ISET
- net Net-(U6-TS/MR) renamed /TSMR
- D5 pad 1: Net-(D5-K) -> /SW
- U1 pad 5: /SD_CLK -> +3v3
Routing:
- added copper zone on B.Cu, net GND
- added copper zone on In1.Cu, net GND
- added copper zone on In2.Cu, net GND
Other:
- board size 39 x 49 mm -> 38 x 44 mm
- copper layers 2 -> 4

Commit message: GS Traces complete
Parts:
- added D7: PWR5, LED_SMD:LED_0805_2012Metric, F.Cu at (225.6, 75.1)
- added G***: LOGO, ESP32 Ground Station:TRT_Logo, B.Cu at (202.4, 107.0)
- added R22: 2k, Resistor_SMD:R_0603_1608Metric, B.Cu at (225.6, 75.1)
- D3: value PWR -> PWR3
- J1: footprint MEM2085:GCT_MEM2085-00-115-00-A_REV0.2 -> MEM2085:microSD-GCT_MEM2085-00-115-00-A_REV0.2
- R13, R15, R16, R17: moved to B.Cu
- U4: moved to F.Cu
- moved D3 23.7 mm to (228.5, 100.7)
- moved R13 20.8 mm to (228.5, 100.6), turned to -90 degrees
- moved R17 10.9 mm to (223.1, 76.1), turned to -90 degrees
- moved R6 10.3 mm to (224.2, 95.8), turned to 180 degrees
- moved C8 10.2 mm to (222.9, 99.9), turned to 0 degrees
- moved R11 8.88 mm to (224.2, 88.2)
- moved D5 8.84 mm to (213.2, 104.0), turned to 90 degrees
- moved R16 8.12 mm to (221.5, 76.1), turned to -90 degrees
- moved D1 7.42 mm to (221.2, 76.1)
- moved D2 7.34 mm to (223.1, 76.1)
- moved R10 6.54 mm to (224.2, 89.8)
- moved R7 6.54 mm to (224.2, 94.2)
- moved R4 6.50 mm to (231.0, 76.5), turned to 90 degrees
- moved R3 6.38 mm to (231.0, 82.9), turned to -90 degrees
- moved C7 6.00 mm to (211.9, 102.8)
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Connections:
- net /DPWR renamed /DPWR3
- J1 pad 5: +3v3 -> /SD_CLK
- U1 pad 5: +3v3 -> /SD_CLK
Routing:
- net GND: track 0.00 -> 135.5 mm, vias 0 -> 64
- net /BAT_STAT_2: track 0.00 -> 90.6 mm, vias 0 -> 3
- net +3v3: track 0.00 -> 85.0 mm, vias 0 -> 7
- net /SPI2_MOSI: track 0.00 -> 61.1 mm, vias 0 -> 4
- net /SPI2_SCK: track 0.00 -> 59.6 mm, vias 0 -> 4
- net /SPI2_MISO: track 0.00 -> 55.6 mm, vias 0 -> 3
- net /RAD_BUSY: track 0.00 -> 43.5 mm, vias 0 -> 3
- net VBUS: track 0.00 -> 42.4 mm, vias 0 -> 2
- net /SD_CMD: track 0.00 -> 42.4 mm, vias 0 -> 3
- net /SPI2_CS1: track 0.00 -> 37.3 mm, vias 0 -> 1
- net /SW: track 0.00 -> 34.4 mm
- net /IO16: track 0.00 -> 32.4 mm, vias 0 -> 2
- net /IO0: track 0.00 -> 32.2 mm, vias 0 -> 1
- net /RAD_IO9: track 0.00 -> 29.7 mm, vias 0 -> 1
- net /RAD_IO8: track 0.00 -> 29.5 mm, vias 0 -> 1
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- added copper zone on B.Cu, net +4v5-1
- added copper zone on F.Cu, net GND
- added copper zone on B.Cu, net VBAT
- added copper zone on B.Cu, net VBUS
- removed copper zone on B.Cu, net GND
Other:
- board text added: "0R"
- board text added: "1.0"
- board text added: "100kR"
- board text added: "100nF"
- board text added: "10kR"
- board text added: "10uF"
- board text added: "13kR"
- board text added: "15uH"
- board text added: "1uF"
- board text added: "2kR"
- board text added: "300R"
- board text added: "3V"
- board text added: "470nF"
- board text added: "5.1kR"
- board text added: "5V"
- board text added: "BAT STAT"
- board text added: "BQ25"
- board text added: "D4"
- board text added: "D5"
- board text added: "DNP"
- board text added: "ESP32-S3-MINI-1"
- board text added: "GPIO"
- board text added: "Ground Station Receiver"
- board text added: "REV"
- board text added: "TPS"
- board text added: "TRT"
- board text added: "Terrapin Rocket Team"
- board text added: "UMD"
- board text added: "USB"
- board text added: "University of Maryland"
- board text added: "XC6"
- board text added: "← 10kR →"

Commit message: aadded silk screen to GPIO pins
Routing:
- net /SPI2_SCK: track 59.6 -> 58.9 mm
Other:
- board text added: "3V 3V"
- board text added: "EN MISO"
- board text added: "GND GND"
- board text added: "IO0 MOSI"
- board text added: "IO16 IO48"
- board text added: "RX SCL"
- board text added: "RX1 IO47"
- board text added: "TX SDA"
- board text added: "TX1 SCK"
